Commit message: twitchy has a wrist.

File: launch/urdf/twitchy.urdf (robot description, URDF)
Before this commit: robot twitchy, 5 links, 4 joints
Links:
- added link wrist; visual cylinder length=0.01 radius=0.016
- link end_effector: geometry visual cylinder length=0.01 radius=0.016
Joints:
- removed joint arm2_to_endeffector
- added joint arm2_to_wrist: type revolute, parent arm_link_2, child wrist, origin xyz=0.14 0.0 -0.015, axis 0 1 0, limit lower=-1.7 upper=1.7 effort=1000.0 velocity=0.5
- added joint wrist_to_endeffector: type revolute, parent wrist, child end_effector, origin xyz=0.0 0.0 -0.01, axis 0 0 1, limit lower=-1.57 upper=1.57 effort=1000.0 velocity=0.5

Commit message: this seems to work.

File: launch/urdf/twitchy.urdf (robot description, URDF)
Before this commit: robot twitchy, 6 links, 5 joints
Joints:
- joint arm2_to_wrist: limit lower=-1.7 upper=1.7 effort=1000.0 velocity=0.5 -> lower=-3.1415 upper=3.1415 effort=1000.0 velocity=0.5
- joint wrist_to_endeffector: origin xyz=0.0 0.0 -0.01 -> xyz=0.0 0.0 0.01

Commit message: got a service to record robot positions.

File: launch/urdf/twitchy.urdf (robot description, URDF)
Before this commit: robot twitchy, 6 links, 5 joints
Links:
- added link magnet; visual cylinder length=0.005 radius=0.008
Joints:
- added joint endeffector_to_magnet: type fixed, parent end_effector, child magnet, origin xyz=0.0 0.0 -0.005
- joint wrist_to_endeffector: origin xyz=0.0 0.0 0.01 -> xyz=0.0 0.0 -0.01

Commit message: a quick update to the urdf and rename of launch files.

File: launch/urdf/twitchy.urdf (robot description, URDF)
Before this commit: robot twitchy, 7 links, 6 joints
Joints:
- joint body_to_arm1: limit lower=0 upper=1.7 effort=1000.0 velocity=0.5 -> lower=0 upper=1 effort=1000.0 velocity=0.5
- joint wrist_to_endeffector: origin xyz=0.0 0.0 -0.01 -> xyz=0.0 0.0 0.01 rpy=0 0 0
